File: Riaa.sch (KiCad schematic (older format))
At the start: 46 parts, among them J1 +15V, J2 GND, J3 -15V, J4 +IN, J5 GND, U1 TL071, U2 TL072, U3 TL071, U4 TL071

Commit message: component values
Parts:
- C1, C3, C6, C7: value C -> 100n
- C2, C4, C8, C9: value C -> 1uF
- C5: value C -> 68p
- R1, R8: value R -> 27k
- R10, R26, R27, R3: value R -> 1M
- R11, R4: value R -> 100
- R12, R28, R5: value R -> 1k
- R13, R6: value R -> 3k9
- R14, R7: value R -> 4k7
- R15, R18: value R -> 47k
- R16: value R -> 220
- R17: value R -> 3k3
- R19, R25: value R -> 100k
- R2, R9: value R -> 2k4
- R20, R21: value R -> 1k5
- R22, R23, R24: value R -> 390
Connections:
- net at J3.1 (P1), R8.2, U2.4 (V-): now also U2.4 (V-)
- net at J1.1 (P1), R1.2, U2.8 (V+): now also U2.8 (V+)
Other:
- moved on the sheet: C1, C3, C7, J2, R27, R9

Commit message: pads
Parts:
- removed J1: +15V, symbol CONN_01X01
- removed J2, J5: GND, symbol CONN_01X01
- removed J3: -15V, symbol CONN_01X01
- removed J4: +IN, symbol CONN_01X01
- added J1: power, Connectors:PINHEAD1-3, symbol CONN_01X03
- added J2: in, Connectors:PINHEAD1-2, symbol CONN_01X02
- added J3: out, Connectors:PINHEAD1-2, symbol CONN_01X02
- C1, C3, C5, C6, C7: footprint (none) -> Capacitors_THT:C_Rect_L7.2mm_W2.5mm_P5.00mm_FKS2_FKP2_MKS2_MKP2
- C2, C4, C8, C9: footprint (none) -> Capacitors_THT:C_Rect_L7.2mm_W5.5mm_P5.00mm_FKS2_FKP2_MKS2_MKP2
- R1, R10, R11, R12, R13, R14, R15, R16, R17, R18, R19, R2, R20, R21, R22, R23, R24, R25, R26, R27, R28, R3, R4, R5, R6, R7, R8, R9: footprint (none) -> Resistors_THT:R_Axial_DIN0207_L6.3mm_D2.5mm_P7.62mm_Horizontal
- U1, U2, U3, U4: footprint (none) -> Housings_DIP:DIP-8_W7.62mm
Connections:
- net GND: now also J1.3 (P3), J2.2 (P2), J3.2 (P2); no longer R25.1
- net at R8.2, U2.4 (V-), U2.4 (V-): now also J1.1 (P1)
- net at R1.2, U2.8 (V+), U2.8 (V+): now also J1.2 (P2)
- net at C5.1, R15.2, U1.3 (+): now also J2.1 (P1)
- net at R24.2, R25.2, R26.1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: now also J3.1 (P1)
Other:
- moved on the sheet: R25

Commit message: layout
Connections:
- net GND: now also R25.1
Changed lines of the file:
@@
 	1900 5800 1900 6100
 Wire Wire Line
-	1900 6100 4850 6100
+	4850 6100 1900 6100
 Wire Wire Line
 	2300 6100 2300 5600
@@
 	5900 5500 6650 5500
 Wire Wire Line
-	6350 5800 6350 6000
+	6350 5850 6350 6000
 Wire Wire Line
 	7100 6000 4850 6000

Commit message: decoupling
Parts:
- added C10: 100n, Capacitors_THT:C_Rect_L7.2mm_W2.5mm_P5.00mm_FKS2_FKP2_MKS2_MKP2, symbol C
Connections:
- net at J1.1 (P1), R8.2, U2.4 (V-)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: now also C10.1
- net at J1.2 (P2), R1.2, U2.8 (V+)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: now also C10.2
Changed lines of the file:
@@
 	1300 2050 1500 2050
 Wire Wire Line
-	1300 1550 4100 1550
+	1300 1500 4100 1500
 Wire Wire Line
-	4100 1550 4100 2050
+	4100 1500 4100 2050
 Wire Wire Line
 	3150 2400 5750 2400
 Wire Wire Line
-	3700 2400 3700 1550
-Connection ~ 3700 1550
+	3700 2400 3700 1500
+Connection ~ 3700 1500
 Wire Wire Line
 	1500 2050 1500 1800
@@
 Connection ~ 3700 2400
 Wire Wire Line
-	1300 1550 1300 1950
+	1300 1500 1300 1950
 Wire Wire Line
 	1300 2650 1300 2150
@@
 	6650 5600 6650 6000
 Connection ~ 6650 6000
+$Comp
+L C C10
+U 1 1 5918A004
+P 1900 1650
+F 0 "C10" H 2015 1696 50  0000 L CNN
+F 1 "100n" H 2015 1605 50  0000 L CNN
+F 2 "Capacitors_THT:C_Rect_L7.2mm_W2.5mm_P5.00mm_FKS2_FKP2_MKS2_MKP2" H 1938 1500 50  0001 C CNN
+F 3 "" H 1900 1650 50  0001 C CNN
+	1    1900 1650
+	1    0    0    -1
+$EndComp
+Connection ~ 1900 1800
+Connection ~ 1900 1500
 $EndSCHEMATC

Commit message: 65x30mm
Parts:
- U1, U3, U4: symbol TL071 -> TL071-RESCUE-Riaa
Changed lines of the file:
@@
 EESchema Schematic File Version 2
+LIBS:Riaa-rescue
 LIBS:power
 LIBS:device
@@
 $EndComp
 $Comp
-L TL071 U1
+L TL071-RESCUE-Riaa U1
 U 1 1 590836D0
 P 3200 5250
@@
 $EndComp
 $Comp
-L TL071 U3
+L TL071-RESCUE-Riaa U3
 U 1 1 590837A4
 P 5650 4900
@@
 $EndComp
 $Comp
-L TL071 U4
+L TL071-RESCUE-Riaa U4
 U 1 1 59083810
 P 8300 4400
@@
 	1900 5800 1900 6100
 Wire Wire Line
-	4850 6100 1900 6100
+	1900 6100 4850 6100
 Wire Wire Line
 	2300 6100 2300 5600
